File: kgm-m3-led-base.kicad_sch (KiCad schematic)
At the start: 26 parts, among them J1 Conn_02x06_Counter_Clockwise

Commit message: Redesigned connector, added spacer model
Parts:
- removed J1: Conn_02x06_Counter_Clockwise, Connector_PinHeader_1.27mm:PinHeader_2x06_P1.27mm_Vertical_SMD, symbol Connector_Generic:Conn_02x06_Counter_Clockwise
- added J1, J2: Conn_02x03_Counter_Clockwise, Connector_PinHeader_2.54mm:PinHeader_2x03_P2.54mm_Vertical_SMD, symbol Connector_Generic:Conn_02x03_Counter_Clockwise
Connections:
- net COM: now also J1.3 (Pin_3), J2.3 (Pin_3)
- net at D6.2 (A): now also J2.1 (Pin_1)
- net at D10.2 (A): now also J2.2 (Pin_2)
- net at D7.2 (A): now also J1.6 (Pin_6)
- net at D4.2 (A): now also J2.5 (Pin_5)
- net at D1.2 (A): now also J1.4 (Pin_4)
- net at D3.2 (A): now also J1.5 (Pin_5)
- net at D9.2 (A): now also J1.2 (Pin_2)
- net at D2.2 (A): now also J2.4 (Pin_4)
- net at D8.2 (A): now also J2.6 (Pin_6)
- net at D5.2 (A): now also J1.1 (Pin_1)
Other:
- moved on the sheet: D1, D10, D2, D3, D4, D5, D6, D7, D8, D9, FID1, FID2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
